Commit message: update: new joint limitation

File: ghand5_system/urdf/ghand5_left.urdf (robot description, URDF)
Before this commit: robot ghand5-left, 19 links, 18 joints
Joints:
- joint FF_PIP: limit lower=0 upper=1.74532925199433 effort=0 velocity=0 -> lower=0 upper=1.39626340159546 effort=0 velocity=0
- joint LF_PIP: limit lower=0 upper=1.65806278939461 effort=0 velocity=0 -> lower=0 upper=1.2915436464758 effort=0 velocity=0
- joint MF_PIP: limit lower=0 upper=1.74532925199433 effort=0 velocity=0 -> lower=0 upper=1.5707963267949 effort=0 velocity=0
- joint RF_PIP: limit lower=0 upper=1.74532925199433 effort=0 velocity=0 -> lower=0 upper=1.5707963267949 effort=0 velocity=0

File: ghand5_system/urdf/ghand5_right.urdf (robot description, URDF)
Before this commit: robot ghand5-right, 19 links, 18 joints
Joints:
- joint FF_PIP: limit lower=0 upper=1.74532925199433 effort=0 velocity=0 -> lower=0 upper=1.39626340159546 effort=0 velocity=0
- joint LF_PIP: limit lower=0 upper=1.65806278939461 effort=0 velocity=0 -> lower=0 upper=1.2915436464758 effort=0 velocity=0
- joint MF_PIP: limit lower=0 upper=1.74532925199433 effort=0 velocity=0 -> lower=0 upper=1.5707963267949 effort=0 velocity=0
- joint RF_PIP: limit lower=0 upper=1.74532925199433 effort=0 velocity=0 -> lower=0 upper=1.5707963267949 effort=0 velocity=0

Commit message: update: 增加被动关节与主动关节的线性拟合关系

File: ghand5_system/urdf/ghand5_left.urdf (robot description, URDF)
Before this commit: robot ghand5-left, 19 links, 18 joints
Joints:
- joint FF_DIP: mimic (none) -> joint=FF_PIP multiplier=0.820453298 offset=-0.032725507235168594
- joint LF_DIP: mimic (none) -> joint=LF_PIP multiplier=0.841152165 offset=-0.03862607626264481
- joint MF_DIP: mimic (none) -> joint=MF_PIP multiplier=0.821680553 offset=-0.033279428226727026
- joint RF_DIP: mimic (none) -> joint=RF_PIP multiplier=0.821680553 offset=-0.033279428226727026
- joint Thumb_IP: mimic (none) -> joint=Thumb_MCP multiplier=1.107174665 offset=0.019096537114922627

File: ghand5_system/urdf/ghand5_right.urdf (robot description, URDF)
Before this commit: robot ghand5-right, 19 links, 18 joints
Joints:
- joint FF_DIP: mimic (none) -> joint=FF_PIP multiplier=0.820453298 offset=-0.032725507235168594
- joint LF_DIP: mimic (none) -> joint=LF_PIP multiplier=0.841152165 offset=-0.03862607626264481
- joint MF_DIP: mimic (none) -> joint=MF_PIP multiplier=0.821680553 offset=-0.033279428226727026
- joint RF_DIP: mimic (none) -> joint=RF_PIP multiplier=0.821680553 offset=-0.033279428226727026
- joint Thumb_IP: mimic (none) -> joint=Thumb_MCP multiplier=1.107174665 offset=0.019096537114922627

Commit message: add: joint effort and velocity

File: ghand5_system/urdf/ghand5_left.urdf (robot description, URDF)
Before this commit: robot ghand5-left, 19 links, 18 joints
Joints:
- joint FF_DIP: limit lower=0 upper=1.5707963267949 effort=0 velocity=0 -> lower=0 upper=1.5707963267949 effort=0.03 velocity=2.181662
- joint FF_MCP: limit lower=0 upper=1.5707963267949 effort=0 velocity=0 -> lower=0 upper=1.5707963267949 effort=0.69 velocity=2.234021
- joint FF_MCP_AA: limit lower=-0.174532925199433 upper=0.174532925199433 effort=0 velocity=0 -> lower=-0.174532925199433 upper=0.174532925199433 effort=0.6 velocity=1.151917
- joint FF_PIP: limit lower=0 upper=1.39626340159546 effort=0 velocity=0 -> lower=0 upper=1.39626340159546 effort=0.18 velocity=2.565634
- joint LF_DIP: limit lower=0 upper=1.5707963267949 effort=0 velocity=0 -> lower=0 upper=1.5707963267949 effort=0.02 velocity=2.059489
- joint LF_MCP: limit lower=0 upper=1.5707963267949 effort=0 velocity=0 -> lower=0 upper=1.5707963267949 effort=0.42 velocity=2.268928
- joint LF_PIP: limit lower=0 upper=1.2915436464758 effort=0 velocity=0 -> lower=0 upper=1.2915436464758 effort=0.11 velocity=2.513274
- joint MF_DIP: limit lower=0 upper=1.5707963267949 effort=0 velocity=0 -> lower=0 upper=1.5707963267949 effort=0.03 velocity=2.181662
- joint MF_MCP: limit lower=0 upper=1.5707963267949 effort=0 velocity=0 -> lower=0 upper=1.5707963267949 effort=0.69 velocity=2.234021
- joint MF_PIP: limit lower=0 upper=1.5707963267949 effort=0 velocity=0 -> lower=0 upper=1.5707963267949 effort=0.18 velocity=2.565634
- joint RF_DIP: limit lower=0 upper=1.5707963267949 effort=0 velocity=0 -> lower=0 upper=1.5707963267949 effort=0.03 velocity=2.181662
- joint RF_MCP: limit lower=0 upper=1.5707963267949 effort=0 velocity=0 -> lower=0 upper=1.5707963267949 effort=0.69 velocity=2.234021
- joint RF_PIP: limit lower=0 upper=1.5707963267949 effort=0 velocity=0 -> lower=0 upper=1.5707963267949 effort=0.18 velocity=2.565634
- joint Thumb_IP: limit lower=0 upper=1.5707963267949 effort=0 velocity=0 -> lower=0 upper=1.5707963267949 effort=0.03 velocity=4.24115
- joint Thumb_MCP: limit lower=0 upper=1.15191730631626 effort=0 velocity=0 -> lower=0 upper=1.15191730631626 effort=0.13 velocity=3.525565
- joint Thumb_TMC_AA: limit lower=0.349065850398866 upper=1.5707963267949 effort=0 velocity=0 -> lower=0.349065850398866 upper=1.5707963267949 effort=0.12 velocity=4.18879
- joint Thumb_TMC_FE: limit lower=0 upper=0.872664625997165 effort=0 velocity=0 -> lower=0 upper=0.872664625997165 effort=0.09 velocity=3.141593
- joint Thumb_TMC_PS: limit lower=-0.174532925199433 upper=1.0471975511966 effort=0 velocity=0 -> lower=-0.174532925199433 upper=1.0471975511966 effort=0.15 velocity=4.18879

File: ghand5_system/urdf/ghand5_right.urdf (robot description, URDF)
Before this commit: robot ghand5-right, 19 links, 18 joints
Joints:
- joint FF_DIP: limit lower=0 upper=1.5707963267949 effort=0 velocity=0 -> lower=0 upper=1.5707963267949 effort=0.03 velocity=2.181662
- joint FF_MCP: limit lower=0 upper=1.5707963267949 effort=0 velocity=0 -> lower=0 upper=1.5707963267949 effort=0.69 velocity=2.234021
- joint FF_MCP_AA: limit lower=-0.174532925199433 upper=0.174532925199433 effort=0 velocity=0 -> lower=-0.174532925199433 upper=0.174532925199433 effort=0.6 velocity=1.151917
- joint FF_PIP: limit lower=0 upper=1.39626340159546 effort=0 velocity=0 -> lower=0 upper=1.39626340159546 effort=0.18 velocity=2.565634
- joint LF_DIP: limit lower=0 upper=1.5707963267949 effort=0 velocity=0 -> lower=0 upper=1.5707963267949 effort=0.02 velocity=2.059489
- joint LF_MCP: limit lower=0 upper=1.5707963267949 effort=0 velocity=0 -> lower=0 upper=1.5707963267949 effort=0.42 velocity=2.268928
- joint LF_PIP: limit lower=0 upper=1.2915436464758 effort=0 velocity=0 -> lower=0 upper=1.2915436464758 effort=0.11 velocity=2.513274
- joint MF_DIP: limit lower=0 upper=1.5707963267949 effort=0 velocity=0 -> lower=0 upper=1.5707963267949 effort=0.03 velocity=2.181662
- joint MF_MCP: limit lower=0 upper=1.5707963267949 effort=0 velocity=0 -> lower=0 upper=1.5707963267949 effort=0.69 velocity=2.234021
- joint MF_PIP: limit lower=0 upper=1.5707963267949 effort=0 velocity=0 -> lower=0 upper=1.5707963267949 effort=0.18 velocity=2.565634
- joint RF_DIP: limit lower=0 upper=1.5707963267949 effort=0 velocity=0 -> lower=0 upper=1.5707963267949 effort=0.03 velocity=2.181662
- joint RF_MCP: limit lower=0 upper=1.5707963267949 effort=0 velocity=0 -> lower=0 upper=1.5707963267949 effort=0.69 velocity=2.234021
- joint RF_PIP: limit lower=0 upper=1.5707963267949 effort=0 velocity=0 -> lower=0 upper=1.5707963267949 effort=0.18 velocity=2.565634
- joint Thumb_IP: limit lower=0 upper=1.5707963267949 effort=0 velocity=0 -> lower=0 upper=1.5707963267949 effort=0.03 velocity=4.24115
- joint Thumb_MCP: limit lower=0 upper=1.15191730631626 effort=0 velocity=0 -> lower=0 upper=1.15191730631626 effort=0.13 velocity=3.525565
- joint Thumb_TMC_AA: limit lower=0.349065850398866 upper=1.5707963267949 effort=0 velocity=0 -> lower=0.349065850398866 upper=1.5707963267949 effort=0.12 velocity=4.18879
- joint Thumb_TMC_FE: limit lower=0 upper=0.872664625997165 effort=0 velocity=0 -> lower=0 upper=0.872664625997165 effort=0.09 velocity=3.141593
- joint Thumb_TMC_PS: limit lower=-0.174532925199433 upper=1.0471975511966 effort=0 velocity=0 -> lower=-0.174532925199433 upper=1.0471975511966 effort=0.15 velocity=4.18879
