Commit message: add: passive_joint_relationship

File: ghand_lite1_system/urdf/glite1_left.urdf (robot description, URDF)
Before this commit: robot glite1-left, 12 links, 11 joints
Joints:
- joint FF_IP: mimic joint=FF_MCP multiplier=0.7721 offset=0 -> joint=FF_MCP multiplier=0.7149 offset=0
- joint LF_IP: mimic joint=LF_MCP multiplier=0.772 offset=0 -> joint=LF_MCP multiplier=0.6939 offset=0
- joint MF_IP: mimic joint=MF_MCP multiplier=0.7721 offset=0 -> joint=MF_MCP multiplier=0.7319 offset=0
- joint RF_IP: mimic joint=RF_MCP multiplier=0.7721 offset=0 -> joint=RF_MCP multiplier=0.7149 offset=0
- joint THUMB_MCP: mimic joint=THUMB_TMC_FE multiplier=1.1 offset=0 -> joint=THUMB_TMC_FE multiplier=1.13 offset=0

File: ghand_lite1_system/urdf/glite1_right.urdf (robot description, URDF)
Before this commit: robot glite1-right, 12 links, 11 joints
Joints:
- joint FF_IP: mimic joint=FF_MCP multiplier=0.7721 offset=0 -> joint=FF_MCP multiplier=0.7149 offset=0
- joint LF_IP: mimic joint=LF_MCP multiplier=0.772 offset=0 -> joint=LF_MCP multiplier=0.6939 offset=0
- joint MF_IP: mimic joint=MF_MCP multiplier=0.7721 offset=0 -> joint=MF_MCP multiplier=0.7319 offset=0
- joint RF_IP: mimic joint=RF_MCP multiplier=0.7721 offset=0 -> joint=RF_MCP multiplier=0.7149 offset=0
- joint THUMB_MCP: mimic joint=THUMB_TMC_FE multiplier=1.1 offset=0 -> joint=THUMB_TMC_FE multiplier=1.13 offset=0

Commit message: Update joint limits and simulator parameters for glite1 left and right hands

File: ghand_lite1_system/urdf/glite1_left.urdf (robot description, URDF)
Before this commit: robot glite1-left, 12 links, 11 joints
Joints:
- joint FF_IP: limit lower=0 upper=1.3962 effort=0.16 velocity=2.4 -> lower=0 upper=1.3794 effort=0.16 velocity=2.4; mimic joint=FF_MCP multiplier=0.7149 offset=0 -> joint=FF_MCP multiplier=0.7721 offset=0
- joint FF_MCP: limit lower=0 upper=1.57 effort=0.2 velocity=2.4 -> lower=0 upper=1.789 effort=0.2 velocity=2.4
- joint LF_IP: limit lower=0 upper=1.3962 effort=0.16 velocity=2.4 -> lower=0 upper=1.4014 effort=0.16 velocity=2.4; mimic joint=LF_MCP multiplier=0.6939 offset=0 -> joint=LF_MCP multiplier=0.772 offset=0
- joint LF_MCP: limit lower=0 upper=1.57 effort=0.2 velocity=2.4 -> lower=0 upper=1.8151 effort=0.2 velocity=2.4
- joint MF_IP: limit lower=0 upper=1.3962 effort=0.16 velocity=2.4 -> lower=0 upper=1.3794 effort=0.16 velocity=2.4; mimic joint=MF_MCP multiplier=0.7319 offset=0 -> joint=MF_MCP multiplier=0.7721 offset=0
- joint MF_MCP: limit lower=0 upper=1.57 effort=0.2 velocity=2.4 -> lower=0 upper=1.789 effort=0.2 velocity=2.4
- joint RF_IP: limit lower=0 upper=1.3962 effort=0.16 velocity=2.4 -> lower=0 upper=1.3794 effort=0.16 velocity=2.4; mimic joint=RF_MCP multiplier=0.7149 offset=0 -> joint=RF_MCP multiplier=0.7721 offset=0
- joint RF_MCP: limit lower=0 upper=1.57 effort=0.2 velocity=2.4 -> lower=0 upper=1.789 effort=0.2 velocity=2.4
- joint THUMB_MCP: limit lower=0 upper=0.8727 effort=0.16 velocity=2.4 -> lower=0 upper=0.9563 effort=0.16 velocity=2.4; mimic joint=THUMB_TMC_FE multiplier=1.13 offset=0 -> joint=THUMB_TMC_FE multiplier=1.1 offset=0

File: ghand_lite1_system/urdf/glite1_right.urdf (robot description, URDF)
Before this commit: robot glite1-right, 12 links, 11 joints
Joints:
- joint FF_IP: limit lower=0 upper=1.3962 effort=0.16 velocity=2.4 -> lower=0 upper=1.3794 effort=0.16 velocity=2.4; mimic joint=FF_MCP multiplier=0.7149 offset=0 -> joint=FF_MCP multiplier=0.7721 offset=0
- joint FF_MCP: limit lower=0 upper=1.57 effort=0.2 velocity=2.4 -> lower=0 upper=1.789 effort=0.2 velocity=2.4
- joint LF_IP: limit lower=0 upper=1.3962 effort=0.16 velocity=2.4 -> lower=0 upper=1.4014 effort=0.16 velocity=2.4; mimic joint=LF_MCP multiplier=0.6939 offset=0 -> joint=LF_MCP multiplier=0.772 offset=0
- joint LF_MCP: limit lower=0 upper=1.57 effort=0.2 velocity=2.4 -> lower=0 upper=1.8151 effort=0.2 velocity=2.4
- joint MF_IP: limit lower=0 upper=1.3962 effort=0.16 velocity=2.4 -> lower=0 upper=1.3794 effort=0.16 velocity=2.4; mimic joint=MF_MCP multiplier=0.7319 offset=0 -> joint=MF_MCP multiplier=0.7721 offset=0
- joint MF_MCP: limit lower=0 upper=1.57 effort=0.2 velocity=2.4 -> lower=0 upper=1.789 effort=0.2 velocity=2.4
- joint RF_IP: limit lower=0 upper=1.3962 effort=0.16 velocity=2.4 -> lower=0 upper=1.3794 effort=0.16 velocity=2.4; mimic joint=RF_MCP multiplier=0.7149 offset=0 -> joint=RF_MCP multiplier=0.7721 offset=0
- joint RF_MCP: limit lower=0 upper=1.57 effort=0.2 velocity=2.4 -> lower=0 upper=1.789 effort=0.2 velocity=2.4
- joint THUMB_MCP: limit lower=0 upper=0.8727 effort=0.16 velocity=2.4 -> lower=0 upper=0.9563 effort=0.16 velocity=2.4; mimic joint=THUMB_TMC_FE multiplier=1.13 offset=0 -> joint=THUMB_TMC_FE multiplier=1.1 offset=0
- joint THUMB_TMC_AA: limit lower=0 upper=1.57 effort=0.2 velocity=2.4 -> lower=0 upper=1.5708 effort=0.2 velocity=2.4
